File: 3lbmelty.kicad_pcb (KiCad board)
At the start: 2 copper layers, 128 x 70 mm, 20 parts, among them J1 Esc 2, J2 Amass_XT90-S, J3 Esc 1, Q1 SUM110P06-07L-E3, Q2 2N7002, U1 MCU, U2 Adafruit_H3LIS311_Breakout, U4 RC_RECEIVER, U5 BUCK_CONVERTER

Commit message: new pcb
Parts:
- removed U1: MCU, Adafruit-Eagle-Library.kicad:Adafruit ItsyBitsy 32u4 - 5V 16MHz
- added C1: 0.1uF, SparkFun-Capacitor:C_0603_1608Metric, F.Cu at (140.5, 105.2)
- added C11: 10uF, SparkFun-Capacitor:C_0805_2012Metric, F.Cu at (152.0, 119.5)
- added C12: 10nF, SparkFun-Capacitor:C_0603_1608Metric, F.Cu at (134.2, 114.8)
- added C2: 22pF, Capacitor_SMD:C_0603_1608Metric, F.Cu at (144.0, 122.2)
- added C4: 22pF, Capacitor_SMD:C_0603_1608Metric, F.Cu at (142.2, 122.2)
- added C5: 0.1uF, SparkFun-Capacitor:C_0603_1608Metric, F.Cu at (151.5, 117.0)
- added C6: 0.1uF, SparkFun-Capacitor:C_0603_1608Metric, F.Cu at (140.5, 122.2)
- added C7: 0.1uF, SparkFun-Capacitor:C_0603_1608Metric, F.Cu at (137.8, 105.0)
- added C8: 0.1uF, SparkFun-Capacitor:C_0603_1608Metric, F.Cu at (147.0, 105.2)
- added C9: 0.1uF, SparkFun-Capacitor:C_0603_1608Metric, F.Cu at (134.0, 109.5)
- added D4: USBLC6-4SC6, digikey-footprints:SOT23-6L, F.Cu at (134.0, 123.0)
- added J4: USB_C_Receptacle, SparkFun-Connector:USB-C_16, F.Cu at (125.2, 121.0)
- added R10: 5.1k, SparkFun-Resistor:R_0603_1608Metric, F.Cu at (129.2, 118.8)
- added R6: 22, SparkFun-Resistor:R_0603_1608Metric, F.Cu at (134.0, 113.0)
- added R7: 22, SparkFun-Resistor:R_0603_1608Metric, F.Cu at (134.0, 111.2)
- added R8: 10k, SparkFun-Resistor:R_0603_1608Metric, F.Cu at (138.8, 122.2)
- added R9: 5.1k, SparkFun-Resistor:R_0603_1608Metric, F.Cu at (124.0, 118.8)
- added SW1: SMD_5.2x5.2mm_h1.5mm, SparkFun-Switch:Push_SMD_5.2x5.2mm_h1.9mm, F.Cu at (155.5, 111.5)
- added U6: ATMEGA32U4-AU, digikey-footprints:TQFP-44_10x10mm, F.Cu at (143.0, 113.8)
- added Y1: 16MHz, SparkFun-Clock:Crystal_SMD_2.0x1.6mm, F.Cu at (147.5, 122.5)
- moved C1 14.6 mm to (128.2, 113.0)
- moved D2 9.59 mm to (117.7, 115.0)
- moved R5 9.59 mm to (128.0, 115.2)
Routing:
- net GND: track 239.3 -> 362.0 mm, vias 27 -> 33
- net 5v: track 145.8 -> 215.7 mm, vias 0 -> 6
- net SDA: track 13.8 -> 57.4 mm, vias 0 -> 2
- net D-: track 0.00 -> 32.8 mm, vias 0 -> 2
- net VBUS: track 0.00 -> 31.7 mm, vias 0 -> 2
- net MOTOR_2: track 75.9 -> 105.2 mm
- net Reset: track 0.00 -> 29.1 mm, vias 0 -> 2
- net SCL: track 14.9 -> 44.0 mm, vias 0 -> 2
- net RC3: track 10.4 -> 36.7 mm, vias 0 -> 1
- net D+: track 0.00 -> 25.3 mm, vias 0 -> 2
- net Net-(U6-PC7): track 4.79 -> 23.4 mm, vias 0 -> 2
- net RC2: track 14.5 -> 32.2 mm, vias 0 -> 1
- net RC1: track 24.1 -> 38.7 mm, vias 0 -> 3
- net Net-(U6-XTAL1): track 0.00 -> 9.52 mm
- net Net-(U6-XTAL2): track 0.00 -> 7.27 mm
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
Commit message: fixed small issue with resistor placement
Parts:
- moved R1 16.5 mm to (166.6, 103.0)
- moved R2 16.5 mm to (161.8, 102.8)
Routing:
- net 5v: track 215.7 -> 194.3 mm
- net SCL: track 44.0 -> 55.3 mm
- net SDA: track 57.4 -> 60.5 mm
Changed lines of the file:
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@@
 			(drillshape 0)
 			(scaleselection 1)
-			(outputdirectory "./")
+			(outputdirectory "D:/Downloads/")
 		)
 	)
@@
 	(footprint "SparkFun-Resistor:R_0805_2012Metric"
 		(layer "F.Cu")
-		(at 148 93.75 180)
+		(at 161.8375 102.75 180)
 		(descr "Resistor SMD 0805 (2012 Metric), square (rectangular) end terminal, IPC_7351 nominal, (Body size source: IPC-SM-782 page 72, https://www.pcb-3d.com/wordpress/wp-content/uploads/ipc-sm-782a_amendment_1_and_2.pdf), generated with kicad-footprint-generator")
 		(tags "SparkFun resistor")
@@
 	(footprint "Resistor_SMD:R_0805_2012Metric"
 		(layer "F.Cu")
-		(at 152.75 94 180)
+		(at 166.5875 103 180)
 		(descr "Resistor SMD 0805 (2012 Metric), square (rectangular) end terminal, IPC-7351 nominal, (Body size source: IPC-SM-782 page 72, https://www.pcb-3d.com/wordpress/wp-content/uploads/ipc-sm-782a_amendment_1_and_2.pdf), generated with kicad-footprint-generator")
 		(tags "resistor")
@@
 	(segment
 		(start 182.073959 113.823959)
-		(end 163.25 95)
+		(end 164.625 96.375)
+		(width 0.2)
+		(layer "F.Cu")
+		(net 1)
+	)
+	(segment
+		(start 160.925 102.75)
+		(end 162.024 103.849)
 		(width 0.2)
 		(layer "F.Cu")
@@
 	)
 	(segment
-		(start 151.75 92.25)
-		(end 151.5 92)
-		(width 0.2)
-		(layer "F.Cu")
-		(net 1)
-	)
-	(segment
-		(start 151.8375 94)
-		(end 151.8375 92.3375)
-		(width 0.2)
-		(layer "F.Cu")
-		(net 1)
-	)
-	(segment
-		(start 145.147545 94.352455)
-		(end 145.147545 98.85)
-		(width 0.2)
-		(layer "F.Cu")
-		(net 1)
-	)
-	(segment
 		(start 148.7 116.95)
 		(end 149.55 116.95)
@@
 	)
 	(segment
-		(start 145.75 92)
-		(end 145.75 93.75)
-		(width 0.2)
-		(layer "F.Cu")
-		(net 1)
-	)
-	(segment
-		(start 163.25 92.25)
-		(end 151.75 92.25)
-		(width 0.2)
-		(layer "F.Cu")
-		(net 1)
-	)
-	(segment
 		(start 131.576 108.724)
 		(end 133.999 108.724)
@@
 	)
 	(segment
-		(start 147.0875 93.75)
-		(end 145.75 93.75)
-		(width 0.2)
-		(layer "F.Cu")
-		(net 1)
-	)
-	(segment
 		(start 135.825 110.55)
 		(end 137.3 110.55)
@@
 	)
 	(segment
-		(start 151.5 92)
-		(end 145.75 92)
-		(width 0.2)
-		(layer "F.Cu")
-		(net 1)
-	)
-	(segment
-		(start 145.75 93.75)
-		(end 145.147545 94.352455)
-		(width 0.2)
-		(layer "F.Cu")
-		(net 1)
-	)
-	(segment
 		(start 139 111.25)
 		(end 138.3 110.55)
@@
 	)
 	(segment
-		(start 151.8375 92.3375)
-		(end 151.75 92.25)
-		(width 0.2)
-		(layer "F.Cu")
-		(net 1)
-	)
-	(segment
 		(start 150.675 116.95)
 		(end 150.725 117)
@@
 	)
 	(segment
+		(start 165.675 103)
+		(end 165.675 97.425)
+		(width 0.2)
+		(layer "F.Cu")
+		(net 1)
+	)
+	(segment
 		(start 150.276 116.224)
 		(end 164.974 116.224)
@@
 	)
 	(segment
+		(start 164.826 103.849)
+		(end 165.675 103)
+		(width 0.2)
+		(layer "F.Cu")
+		(net 1)
+	)
+	(segment
 		(start 133.999 108.724)
 		(end 134.775 109.5)
@@
 	)
 	(segment
+		(start 162.024 103.849)
+		(end 164.826 103.849)
+		(width 0.2)
+		(layer "F.Cu")
+		(net 1)
+	)
+	(segment
 		(start 147 106.025)
 		(end 147 108.05)
@@
 	)
 	(segment
-		(start 163.25 95)
-		(end 163.25 92.25)
-		(width 0.2)
-		(layer "F.Cu")
-		(net 1)
-	)
-	(segment
 		(start 138 107.25)
 		(end 138.2 107.25)
@@
 	)
 	(segment
-		(start 153.6625 94)
-		(end 153.6625 97.204955)
+		(start 166.25 104.25)
+		(end 167.5 103)
+		(width 0.2)
+		(layer "F.Cu")
+		(net 11)
+	)
+	(segment
+		(start 159.43 104.25)
+		(end 166.25 104.25)
 		(width 0.2)
 		(layer "F.Cu")
@@
 	)
 	(segment
-		(start 159.43 102.972456)
+		(start 159.43 104.25)
 		(end 159.43 105.38)
 		(width 0.2)
@@
 	)
 	(segment
-		(start 144.75 119.3)
-		(end 144.6 119.45)
+		(start 159.43 102.972456)
+		(end 159.43 104.25)
 		(width 0.2)
 		(layer "F.Cu")
@@
 	)
 	(segment
-		(start 153.6625 97.204955)
-		(end 155.307545 98.85)
+		(start 144.75 119.3)
+		(end 144.6 119.45)
 		(width 0.2)
 		(layer "F.Cu")
@@
 	)
 	(segment
-		(start 148.9125 93.75)
-		(end 148.9125 94.994955)
+		(start 154.208773 100.291227)
+		(end 154.117545 100.199999)
+		(width 0.2)
+		(layer "F.Cu")
+		(net 12)
+	)
+	(segment
+		(start 163.774545 101.725455)
+		(end 162.75 102.75)
+		(width 0.2)
+		(layer "F.Cu")
+		(net 12)
+	)
+	(segment
+		(start 154.117545 98.357085)
+		(end 155.740402 96.734228)
+		(width 0.2)
+		(layer "F.Cu")
+		(net 12)
+	)
+	(segment
+		(start 154.208773 100.291227)
+		(end 152.767545 98.85)
+		(width 0.2)
+		(layer "F.Cu")
+		(net 12)
+	)
+	(segment
+		(start 162.531757 96.734228)
+		(end 163.774545 97.977016)
 		(width 0.2)
 		(layer "F.Cu")
@@
 	(segment
 		(start 156.89 102.972455)
-		(end 152.767545 98.85)
+		(end 154.208773 100.291227)
 		(width 0.2)
 		(layer "F.Cu")
@@
 	)
 	(segment
+		(start 163.774545 97.977016)
+		(end 163.774545 101.725455)
+		(width 0.2)
+		(layer "F.Cu")
+		(net 12)
+	)
+	(segment
 		(start 156.89 105.38)
 		(end 156.89 102.972455)
@@
 	)
 	(segment
-		(start 148.9125 94.994955)
-		(end 152.767545 98.85)
+		(start 154.117545 100.199999)
+		(end 154.117545 98.357085)
 		(width 0.2)
 		(layer "F.Cu")
@@
 		(width 0.2)
 		(layer "F.Cu")
+		(net 12)
+	)
+	(segment
+		(start 155.740402 96.734228)
+		(end 162.531757 96.734228)
+		(width 0.2)
+		(layer "F.Cu")
